File: rectangle-clock/rectangle-clock.kicad_pcb (KiCad board)
At the start: 2 copper layers, 140 x 90 mm, 4 parts

Commit message: update
Parts:
- added BT1: Battery_Cell, footprints:BatteryHolder_Keystone_106_1x20mm, F.Cu at (97.0, 99.4)
- added C1: C_0805_0.1uf, footprints:C_0805_2012Metric, F.Cu at (153.4, 125.0)
- added C2: C_0805_0.1uf, footprints:C_0805_2012Metric, F.Cu at (157.5, 125.0)
- added C3: C_22pf, footprints:C_0805_2012Metric, F.Cu at (154.0, 139.4)
- added C4: C_22pf, footprints:C_0805_2012Metric, F.Cu at (174.3, 139.4)
- added C5: C_0805_1uf, footprints:C_0805_2012Metric, F.Cu at (188.4, 128.0)
- added C6: C_0.1uf, footprints:C_0805_2012Metric, F.Cu at (200.7, 114.3)
- added C7: C_0805_0.1uf, footprints:C_0805_2012Metric, F.Cu at (188.4, 131.3)
- added D1: LED_0805_GRN, footprints:LED_0805_2012Metric, F.Cu at (143.5, 141.2)
- added DS1: Display 1, footprints:Adafruit-1001-0-0-MFG, F.Cu at (147.6, 73.0)
- added DS2: Display 2, footprints:Adafruit-1001-0-0-MFG, F.Cu at (147.6, 93.7)
- added J1: PJ-102AH, footprints:PJ-102AH, F.Cu at (206.7, 129.5)
- added J2: Conn_01x06, footprints:PinHeader_1x06_P2.54mm_Vertical, F.Cu at (213.4, 101.6)
- added J3: Conn_01x07, footprints:PinHeader_1x07_P2.54mm_Vertical, F.Cu at (113.5, 139.7)
- added R1: R_10K, footprints:R_0805_2012Metric, F.Cu at (134.9, 123.2)
- added R10: R_0805_4.7K, footprints:R_0805_2012Metric, F.Cu at (205.7, 111.8)
- added R11: R_0805_4.7K, footprints:R_0805_2012Metric, F.Cu at (205.7, 109.2)
- added R12: R_0805_1K, footprints:R_0805_2012Metric, F.Cu at (160.0, 114.6)
- added R13: R_2.2K, footprints:R_0805_2012Metric, F.Cu at (143.5, 138.2)
- added R2: R_0805_10K, footprints:R_0805_2012Metric, F.Cu at (191.8, 96.5)
- added R3: R_10K, footprints:R_0805_2012Metric, F.Cu at (137.4, 123.2)
- added R4: R_10K, footprints:R_0805_2012Metric, F.Cu at (177.8, 114.3)
- added R5: R_0805_1K, footprints:R_0805_2012Metric, F.Cu at (107.7, 124.5)
- added R6: R_0805_1K, footprints:R_0805_2012Metric, F.Cu at (139.7, 59.4)
- added R7: PhotoconductivePhotocell, footprints:R_LDR_4.9x4.2mm_P2.54mm_Vertical, F.Cu at (150.0, 59.9)
- added R8: R_0805_1K, footprints:R_0805_2012Metric, F.Cu at (125.2, 114.3)
- added R9: R_0805_1K, footprints:R_0805_2012Metric, F.Cu at (142.7, 114.6)
- added SW1: Omron_B3F_SPST, footprints:SW_SPST_Omron_B3FS-100xP, F.Cu at (188.0, 111.8)
- added SW2: Omron_B3F_SPST, footprints:SW_SPST_Omron_B3FS-100xP, F.Cu at (132.8, 116.8)
- added SW3: Omron_B3F_SPST, footprints:SW_SPST_Omron_B3FS-100xP, F.Cu at (150.4, 117.1)
- added SW4: Omron_B3F_SPST, footprints:SW_SPST_Omron_B3FS-100xP, F.Cu at (167.6, 117.1)
- added U1: ATmega328-PU, footprints:DIP-28_W7.62mm, F.Cu at (134.9, 134.9)
- added U2: L7805_TO92, footprints:TO-92_Inline, F.Cu at (196.3, 131.0)
- added U3: MAX7219, footprints:DIP-24_W7.62mm, F.Cu at (207.0, 84.8)
- added U4: DS1307_DIP-8, footprints:DIP-8_W7.62mm, F.Cu at (121.7, 127.8)
- added Y1: Crystal_16MHz, footprints:Crystal_SMD_HC49-SD, F.Cu at (164.2, 139.4)
- added Y2: Crystal_32768Hz, footprints:Crystal_SMD_2Pin_3.2x1.5mm, F.Cu at (118.6, 129.0)
Routing:
- net SEGB: track 0.00 -> 134.5 mm
- net SEGF: track 0.00 -> 119.3 mm
- net PHR: track 0.00 -> 117.4 mm
- net RXD: track 0.00 -> 108.4 mm
- net SEGA: track 0.00 -> 105.5 mm
- net SEGD: track 0.00 -> 94.9 mm
- net Din: track 0.00 -> 94.5 mm
- net SEGE: track 0.00 -> 93.0 mm
- net TXD: track 0.00 -> 89.9 mm
- net SEGDP: track 0.00 -> 89.2 mm
- net RESET: track 0.00 -> 87.5 mm
- net DIG3: track 0.00 -> 83.6 mm
- net SEGC: track 0.00 -> 81.1 mm
- net DIG0: track 0.00 -> 74.4 mm
- net SEGG: track 0.00 -> 70.6 mm
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- added copper zone on B.Cu, net GND
- added copper zone on F.Cu, net VCC
